Commit message: Adding krytn with more detail

File: robot_description/krytn/krytn.urdf.xacro (robot description, xacro)
@@ -1,59 +1,186 @@
 <?xml version='1.0' encoding='utf-8'?>
 <robot xmlns:xacro="http://www.ros.org/wiki/xacro" name="krytn">
-<!-- Set this variable to True to setup for use with Gazebo simulation. -->
-<xacro:arg name="gazebo" default="True" />
-<!-- Import and add robot components -->
-<xacro:include filename="$(find krytn)/robot_description/magni/magni.urdf.xacro" />
-<!-- Configure Control of Joints -->
-<ros2_control name="magni" type="system">
-        <xacro:if value="${$(arg gazebo) == True}">
-                <hardware>
-                        <plugin>ign_ros2_control/IgnitionSystem</plugin>
-                </hardware>
-        </xacro:if>
-        <xacro:if value="${not $(arg gazebo)}">
-                <hardware>
-                        <plugin>ubiquity_motor/UbiquityMotorSystemHardware</plugin>
-                        <param name="serial_port">/dev/serial0</param>
-                        <param name="baud_rate">38400</param>
-                        <param name="left_wheel_joint_name">left_wheel_joint</param>
-                        <param name="right_wheel_joint_name">right_wheel_joint</param>
-                </hardware>
-                <gpio name="magni_IOs">
-                        <state_interface name="battery_voltage"/>
-                </gpio>
-        </xacro:if>
-        <joint name="left_wheel_joint">
-                <command_interface name="velocity">
-                        <param name="min">-1</param>
-                        <param name="max">1</param>
-                </command_interface>
-                <state_interface name="position"/>
-                <state_interface name="velocity"/>
-        </joint>
-        <joint name="right_wheel_joint">
-                <command_interface name="velocity">
-                        <param name="min">-1</param>
-                        <param name="max">1</param>
-                </command_interface>
-                <state_interface name="position"/>
-                <state_interface name="velocity"/>
-        </joint>
-</ros2_control>
-<!-- Setup Gazebo plugins -->
-<xacro:if value="$(arg gazebo)">
+  <!-- Set this variable to True to setup for use with Gazebo simulation. -->
+  <xacro:arg name="gazebo" default="True" />
+  <!-- Import and add robot components -->
+  <xacro:include filename="$(find krytn)/robot_description/magni/magni.urdf.xacro" />
+  <xacro:include filename="$(find realsense2_description)/urdf/_d435i.urdf.xacro" />
+  <!-- Including realsense description from external package -->
+  <xacro:sensor_d435i parent="base_link" name="sensor_d435i" use_nominal_extrinsics="$(arg gazebo)">
+    <origin xyz="0 0 0.3" rpy="0 0 0"/>
+  </xacro:sensor_d435i>
+  <!-- Adding a simple rplidar for collision avoidance.  -->
+  <link name="rplidar">
+    <xacro:cylinder_inertial_with_origin radius="0.02" length="0.35" mass="0.13">
+      <origin xyz="0 0 0.03" rpy="0 ${pi/2} 0" />
+    </xacro:cylinder_inertial_with_origin>
+    <collision name="collision_base">
+      <pose>0 0 0.0175015175 0 0 0</pose>
+      <geometry>
+        <box size="0.05001062 0.05001062 0.035003035"/>
+      </geometry>
+    </collision>
+    <collision name="collision_top">
+      <pose>0 0 0.0525045525 0 0 0</pose>
+      <geometry>
+        <cylinder radius="0.02" length="0.035003035" />
+      </geometry>
+    </collision>
+    <visual name="visual">
+      <pose>0 0 0 0 0 1.5707</pose>
+      <geometry>
+        <mesh filename="file://$(find krytn)/robot_description/krytn/meshes/lidar_2d_v1.dae"/>
+      </geometry>
+    </visual>
+  </link>
+  <joint name="rplidar_joint" type="fixed">
+    <parent link="base_link"/>
+    <child link="rplidar"/>
+    <origin xyz="-0.093 0 0.158" rpy="0 0 0"/>
+  </joint>
+  <!-- Configure Control of Joints -->
+  <ros2_control name="magni" type="system">
+    <xacro:if value="${$(arg gazebo) == True}">
+      <hardware>
+        <plugin>ign_ros2_control/IgnitionSystem</plugin>
+      </hardware>
+    </xacro:if>
+    <xacro:if value="${not $(arg gazebo)}">
+      <hardware>
+        <plugin>ubiquity_motor/UbiquityMotorSystemHardware</plugin>
+        <param name="serial_port">/dev/serial0</param>
+        <param name="baud_rate">38400</param>
+        <param name="left_wheel_joint_name">left_wheel_joint</param>
+        <param name="right_wheel_joint_name">right_wheel_joint</param>
+      </hardware>
+      <gpio name="magni_IOs">
+        <state_interface name="battery_voltage"/>
+      </gpio>
+    </xacro:if>
+    <joint name="left_wheel_joint">
+      <command_interface name="velocity">
+        <param name="min">-1</param>
+        <param name="max">1</param>
+      </command_interface>
+      <state_interface name="position"/>
+      <state_interface name="velocity"/>
+    </joint>
+    <joint name="right_wheel_joint">
+      <command_interface name="velocity">
+        <param name="min">-1</param>
+        <param name="max">1</param>
+      </command_interface>
+      <state_interface name="position"/>
+      <state_interface name="velocity"/>
+    </joint>
+  </ros2_control>
+  <!-- Setup Gazebo plugins -->
+  <xacro:if value="$(arg gazebo)">
     <gazebo>
-        <plugin filename="ign_ros2_control-system" name="ign_ros2_control::IgnitionROS2ControlPlugin">
-                <ros>
-                        <remapping>/diff_drive_base_controller/odometry:=odom</remapping>
-                        <remapping>/diff_drive_base_controller/tf_odometry:=tf</remapping>
-                        <remapping>/diff_drive_base_controller/cmd_vel_unstamped:=cmd_vel</remapping>
-                </ros>
-                <parameters>$(find krytn)/config/diffdrive_control.yaml</parameters>
-        </plugin>
-        <plugin filename="ignition-gazebo-sensors-system" name="ignition::gazebo::systems::Sensors">
-                <render_engine>ogre2</render_engine>
-        </plugin>
+      <plugin filename="ign_ros2_control-system" name="ign_ros2_control::IgnitionROS2ControlPlugin">
+        <ros>
+          <remapping>/diff_drive_base_controller/odometry:=odom</remapping>
+          <remapping>/diff_drive_base_controller/tf_odometry:=tf</remapping>
+          <remapping>/diff_drive_base_controller/cmd_vel_unstamped:=cmd_vel</remapping>
+        </ros>
+        <parameters>$(find krytn)/config/diffdrive_control.yaml</parameters>
+      </plugin>
+      <plugin filename="ignition-gazebo-imu-system" name="gz::sim::systems::Imu">
+      </plugin>
+      <plugin filename="ignition-gazebo-sensors-system" name="ignition::gazebo::systems::Sensors">
+        <render_engine>ogre2</render_engine>
+      </plugin>
     </gazebo>
-</xacro:if>
+    <!-- Add sensor tags to Realsense links -->
+    <gazebo reference="sensor_d435i">
+      <sensor name="realsense_d435" type="rgbd_camera">
+        <topic>realsense</topic>
+        <ignition_frame_id>realsense_d435</ignition_frame_id>
+        <update_rate>5</update_rate>
+        <camera name="camera">
+          <horizontal_fov>0.5</horizontal_fov>
+          <lens>
+            <intrinsics>
+              <!-- fx = fy = width / ( 2 * tan (hfov / 2 ) ) -->
+              <fx>554.25469</fx>
+              <fy>554.25469</fy>
+              <!-- cx = ( width + 1 ) / 2 -->
+              <cx>320.5</cx>
+              <!-- cy = ( height + 1 ) / 2 -->
+              <cy>240.5</cy>
+              <s>0</s>
+            </intrinsics>
+          </lens>
+          <distortion>
+            <k1>0.0</k1>
+            <k2>0.0</k2>
+            <k3>0.0</k3>
+            <p1>0.0</p1>
+            <p2>0.0</p2>
+            <center>0.5 0.5</center>
+          </distortion>
+          <image>
+            <width>160</width>
+            <height>120</height>
+            <format>R8G8B8</format>
+          </image>
+          <clip>
+            <near>0.01</near>
+            <far>10</far>
+          </clip>
+          <depth_camera>
+            <clip>
+              <near>0.1</near>
+              <far>10</far>
+            </clip>
+          </depth_camera>
+          <noise>
+            <type>gaussian</type>
+            <mean>0</mean>
+            <stddev>0.007</stddev>
+          </noise>
+        </camera>
+      </sensor>
+    </gazebo>
+    <gazebo reference="sensor_d435i_accel_frame">
+      <sensor name="imu" type="imu">
+        <always_on>1</always_on>
+        <update_rate>100</update_rate>
+        <visualize>true</visualize>
+        <topic>imu</topic>
+        <enable_metrics>true</enable_metrics>
+      </sensor>
+    </gazebo>
+    <!-- Add sensor tag to Lidar -->
+    <gazebo reference="rplidar">
+      <sensor name="lidar_2d_v1" type="gpu_ray">
+        <topic>lidar</topic>
+        <ignition_frame_id>lidar_2d_v1</ignition_frame_id>
+        <pose>0 0 0.0525045525 0 0 0</pose>
+        <ray>
+          <scan>
+            <horizontal>
+              <samples>90</samples>
+              <resolution>1</resolution>
+              <min_angle>-1.41</min_angle>
+              <max_angle>1.41</max_angle>
+            </horizontal>
+          </scan>
+          <range>
+            <min>0.060</min>
+            <max>10</max>
+            <resolution>0.04</resolution>
+          </range>
+          <noise>
+            <type>gaussian</type>
+            <mean>0.0</mean>
+            <stddev>0.001</stddev>
+          </noise>
+        </ray>
+        <always_on>0</always_on>
+        <update_rate>20</update_rate>
+        <visualize>false</visualize>
+      </sensor>
+    </gazebo>
+  </xacro:if>
 </robot>

Commit message: Minor changes. Unlimited wheel velocity so krytn moves faster!

File: robot_description/krytn/krytn.urdf.xacro (robot description, xacro)
@@ -60,17 +60,19 @@
     <joint name="left_wheel_joint">
       <command_interface name="velocity">
-        <param name="min">-1</param>
-        <param name="max">1</param>
+        <param name="min">-10</param>
+        <param name="max">10</param>
       </command_interface>
       <state_interface name="position"/>
       <state_interface name="velocity"/>
+      <state_interface name="effort" />
     </joint>
     <joint name="right_wheel_joint">
       <command_interface name="velocity">
-        <param name="min">-1</param>
-        <param name="max">1</param>
+        <param name="min">-10</param>
+        <param name="max">10</param>
       </command_interface>
       <state_interface name="position"/>
       <state_interface name="velocity"/>
+      <state_interface name="effort" />
     </joint>
   </ros2_control>
@@ -93,11 +95,11 @@
     </gazebo>
     <!-- Add sensor tags to Realsense links -->
-    <gazebo reference="sensor_d435i">
+    <gazebo reference="sensor_d435i_link">
       <sensor name="realsense_d435" type="rgbd_camera">
         <topic>realsense</topic>
-        <ignition_frame_id>realsense_d435</ignition_frame_id>
+        <ignition_frame_id>sensor_d435i_link</ignition_frame_id>
         <update_rate>5</update_rate>
         <camera name="camera">
-          <horizontal_fov>0.5</horizontal_fov>
+          <horizontal_fov>${86/180}</horizontal_fov>
           <lens>
             <intrinsics>
@@ -156,19 +158,19 @@
       <sensor name="lidar_2d_v1" type="gpu_ray">
         <topic>lidar</topic>
-        <ignition_frame_id>lidar_2d_v1</ignition_frame_id>
+        <ignition_frame_id>rplidar</ignition_frame_id>
         <pose>0 0 0.0525045525 0 0 0</pose>
         <ray>
           <scan>
             <horizontal>
-              <samples>90</samples>
+              <samples>180</samples>
               <resolution>1</resolution>
-              <min_angle>-1.41</min_angle>
-              <max_angle>1.41</max_angle>
+              <min_angle>${-pi}</min_angle>
+              <max_angle>${pi}</max_angle>
             </horizontal>
           </scan>
           <range>
-            <min>0.060</min>
-            <max>10</max>
-            <resolution>0.04</resolution>
+            <min>0.06</min>
+            <max>5</max>
+            <resolution>0.01</resolution>
           </range>
           <noise>

File: robot_description/magni/magni.urdf.xacro (robot description, xacro)
@@ -5,28 +5,28 @@
   <xacro:include filename="$(find krytn)/robot_description/magni/inertial.xacro" />
   <xacro:macro name="low_friction">
-              <mu>0.1</mu>
-              <mu1>0.1</mu1>
-              <mu2>0.1</mu2>
-              <slip1>0</slip1>
-              <slip2>0</slip2>
+    <mu>0.1</mu>
+    <mu1>0.1</mu1>
+    <mu2>0.1</mu2>
+    <slip1>0</slip1>
+    <slip2>0</slip2>
   </xacro:macro>
   <xacro:macro name="high_friction">
-      <collision>
-        <surface>
-          <friction>
-            <ode>
-              <mu>1.0</mu>
-              <mu2>1.0</mu2>
-              <fdir1>0 0 1</fdir1>
-              <slip1>0.0</slip1>
-              <slip2>0.0</slip2>
-              <min_depth>0.001</min_depth>
-              <kp>1e8</kp>
-            </ode>
-          </friction>
-        </surface>
-      </collision>
+    <collision>
+      <surface>
+        <friction>
+          <ode>
+            <mu>1.0</mu>
+            <mu2>1.0</mu2>
+            <fdir1>0 0 1</fdir1>
+            <slip1>0.0</slip1>
+            <slip2>0.0</slip2>
+            <min_depth>0.001</min_depth>
+            <kp>1e8</kp>
+          </ode>
+        </friction>
+      </surface>
+    </collision>
   </xacro:macro>
- <link name="base_footprint"/>
+  <link name="base_footprint"/>
   <joint name="base_footprint_joint" type="fixed">
     <parent link="base_footprint"/>
@@ -44,5 +44,5 @@
     </visual>
     <collision>
-	    <origin xyz="${-wheel_xpos} 0 ${-wheel_r+0.151}" rpy="0 0 0" />
+      <origin xyz="${-wheel_xpos} 0 ${-wheel_r+0.151}" rpy="0 0 0" />
       <geometry>
         <box size="0.398 0.268 0.160"/>
@@ -67,12 +67,12 @@
       </geometry>
     </collision>
-    <xacro:box_inertial_with_origin  x="0.398" y="0.221" z="0.150" mass="10.0">
+    <xacro:box_inertial_with_origin x="0.398" y="0.221" z="0.150" mass="10.0">
       <origin xyz="-0.15 0 0.03" rpy="0 0 0" />
     </xacro:box_inertial_with_origin>
   </link>
   <gazebo reference="base_link">
-  <xacro:low_friction/>
+    <xacro:low_friction/>
   </gazebo>
- <!-- Macro for defining wheels -->
+  <!-- Macro for defining wheels -->
   <xacro:macro name="wheel" params="prefix reflect">
     <link name="${prefix}_wheel">
@@ -99,7 +99,8 @@
       <origin xyz="0 ${0.163*reflect} 0" rpy="0 0 ${pi/2}"/>
       <dynamics damping="0.2" friction="0.8"/>
+      <limit effort="1000" velocity="10" stiffness="0" dissipation="0"/>
     </joint>
     <gazebo reference="${prefix}_wheel">
-    <xacro:high_friction/>
+      <xacro:high_friction/>
     </gazebo>
   </xacro:macro>
@@ -128,9 +129,9 @@
       <child link="${prefix}_caster_wheel"/>
     </joint>
-  <gazebo reference="${prefix}_caster_wheel">
-     <xacro:low_friction/>
-  </gazebo>
+    <gazebo reference="${prefix}_caster_wheel">
+      <xacro:low_friction/>
+    </gazebo>
   </xacro:macro>
-    <!-- and caster wheels )-->
+  <!-- and caster wheels )-->
   <xacro:caster_wheel prefix="left" reflect="1"/>
   <xacro:caster_wheel prefix="right" reflect="-1"/>

Commit message: Adding solutions for localization and adding a tray

File: robot_description/krytn/krytn.urdf.xacro (robot description, xacro)
@@ -8,5 +8,5 @@
   <!-- Including realsense description from external package -->
   <xacro:sensor_d435i parent="base_link" name="sensor_d435i" use_nominal_extrinsics="$(arg gazebo)">
-    <origin xyz="0 0 0.3" rpy="0 0 0"/>
+    <origin rpy="0.0 -0.0 0.0" xyz="0.02 0.0 0.435"/>
   </xacro:sensor_d435i>
   <!-- Adding a simple rplidar for collision avoidance.  -->
@@ -188,3 +188,15 @@
     </gazebo>
   </xacro:if>
+  <link name="tray_link">
+    <visual name="visual">
+      <geometry>
+        <mesh filename="file://$(find krytn)/robot_description/krytn/meshes/tray.dae"/>
+      </geometry>
+    </visual>
+  </link>
+  <joint name="tray_joint" type="fixed">
+    <parent link="base_link"/>
+    <child link="tray_link"/>
+    <origin rpy="0.0 -0.0 0.0" xyz="0.03 0.0 0.25"/>
+  </joint>
 </robot>

Commit message: Setup for jazzy, moving away from setup.py towards CMakeLists build

File: robot_description/krytn/krytn.urdf.xacro (robot description, xacro)
@@ -10,4 +10,11 @@
     <origin xyz="0 0 0.3" rpy="0 0 0"/>
   </xacro:sensor_d435i>
+  <gazebo reference="sensor_d435i_link">
+    <visual>
+      <geometry>
+        <mesh filename="package://realsense2_description/meshes/d435.dae" />
+      </geometry>
+    </visual>
+  </gazebo>
   <!-- Adding a simple rplidar for collision avoidance.  -->
   <link name="rplidar">
@@ -83,7 +90,7 @@
         <controller_manager_prefix_node_name>/krytn</controller_manager_prefix_node_name>
         <ros>
-          <remapping>diff_drive_base_controller/odometry:=odom</remapping>
-          <remapping>diff_drive_base_controller/tf_odometry:=tf</remapping>
-          <remapping>diff_drive_base_controller/cmd_vel_unstamped:=cmd_vel</remapping>
+          <remapping>/krytn/diff_drive_base_controller/odometry:=odom</remapping>
+          <remapping>/krytn/diff_drive_base_controller/tf_odometry:=tf</remapping>
+          <remapping>/krytn/diff_drive_base_controller/cmd_vel_unstamped:=cmd_vel</remapping>
           <namespace>/krytn</namespace>
         </ros>
@@ -100,5 +107,5 @@
       <sensor name="realsense_d435" type="rgbd_camera">
         <topic>realsense</topic>
-        <ignition_frame_id>sensor_d435i_link</ignition_frame_id>
+        <gazebo_frame_id>sensor_d435i_link</gazebo_frame_id>
         <update_rate>5</update_rate>
         <camera name="camera">
@@ -160,5 +167,5 @@
       <sensor name="lidar_2d_v1" type="gpu_ray">
         <topic>lidar</topic>
-        <ignition_frame_id>rplidar</ignition_frame_id>
+        <gazebo_frame_id>rplidar</gazebo_frame_id>
         <pose>0 0 0.0525045525 0 0 0</pose>
         <ray>

File: robot_description/magni/magni.urdf.xacro (robot description, xacro)
@@ -5,9 +5,15 @@
   <xacro:include filename="$(find krytn)/robot_description/magni/inertial.xacro" />
   <xacro:macro name="low_friction">
-    <mu>0.1</mu>
-    <mu1>0.1</mu1>
-    <mu2>0.1</mu2>
-    <slip1>0</slip1>
-    <slip2>0</slip2>
+    <collision>
+      <surface>
+        <friction>
+          <mu>0.1</mu>
+          <mu1>0.1</mu1>
+          <mu2>0.1</mu2>
+          <slip1>0</slip1>
+          <slip2>0</slip2>
+        </friction>
+      </surface>
+    </collision>
   </xacro:macro>
   <xacro:macro name="high_friction">
@@ -21,6 +27,4 @@
             <slip1>0.0</slip1>
             <slip2>0.0</slip2>
-            <min_depth>0.001</min_depth>
-            <kp>1e8</kp>
           </ode>
         </friction>

Commit message: Revert "Jazzy"

File: robot_description/krytn/krytn.urdf.xacro (robot description, xacro)
@@ -10,11 +10,4 @@
     <origin xyz="0 0 0.3" rpy="0 0 0"/>
   </xacro:sensor_d435i>
-  <gazebo reference="sensor_d435i_link">
-    <visual>
-      <geometry>
-        <mesh filename="package://realsense2_description/meshes/d435.dae" />
-      </geometry>
-    </visual>
-  </gazebo>
   <!-- Adding a simple rplidar for collision avoidance.  -->
   <link name="rplidar">
@@ -47,8 +40,8 @@
   </joint>
   <!-- Configure Control of Joints -->
-  <ros2_control name="Krytn" type="system">
+  <ros2_control name="magni" type="system">
     <xacro:if value="${$(arg gazebo) == True}">
       <hardware>
-        <plugin>gz_ros2_control/GazeboSimSystem</plugin>
+        <plugin>ign_ros2_control/IgnitionSystem</plugin>
       </hardware>
     </xacro:if>
@@ -85,17 +78,17 @@
   <xacro:if value="$(arg gazebo)">
     <gazebo>
-      <plugin filename="gz_ros2_control-system" name="gz_ros2_control::GazeboSimROS2ControlPlugin">
+      <plugin filename="ign_ros2_control-system" name="ign_ros2_control::IgnitionROS2ControlPlugin">
         <controller_manager_prefix_node_name>/krytn</controller_manager_prefix_node_name>
         <ros>
-          <remapping>/krytn/diff_drive_base_controller/odometry:=odom</remapping>
-          <remapping>/krytn/diff_drive_base_controller/tf_odometry:=tf</remapping>
-          <remapping>/krytn/diff_drive_base_controller/cmd_vel_unstamped:=cmd_vel</remapping>
+          <remapping>diff_drive_base_controller/odometry:=odom</remapping>
+          <remapping>diff_drive_base_controller/tf_odometry:=tf</remapping>
+          <remapping>diff_drive_base_controller/cmd_vel_unstamped:=cmd_vel</remapping>
           <namespace>/krytn</namespace>
         </ros>
         <parameters>$(find krytn)/config/diffdrive_control.yaml</parameters>
       </plugin>
-      <plugin filename="gz-sim-imu-system" name="gz::sim::systems::Imu">
+      <plugin filename="ignition-gazebo-imu-system" name="gz::sim::systems::Imu">
       </plugin>
-      <plugin filename="gz-sim-sensors-system" name="gz::sim::systems::Sensors">
+      <plugin filename="ignition-gazebo-sensors-system" name="ignition::gazebo::systems::Sensors">
         <render_engine>ogre2</render_engine>
       </plugin>
@@ -105,5 +98,5 @@
       <sensor name="realsense_d435" type="rgbd_camera">
         <topic>realsense</topic>
-        <gazebo_frame_id>sensor_d435i_link</gazebo_frame_id>
+        <ignition_frame_id>sensor_d435i_link</ignition_frame_id>
         <update_rate>5</update_rate>
         <camera name="camera">
@@ -165,5 +158,5 @@
       <sensor name="lidar_2d_v1" type="gpu_ray">
         <topic>lidar</topic>
-        <gazebo_frame_id>rplidar</gazebo_frame_id>
+        <ignition_frame_id>rplidar</ignition_frame_id>
         <pose>0 0 0.0525045525 0 0 0</pose>
         <ray>

File: robot_description/magni/magni.urdf.xacro (robot description, xacro)
@@ -5,15 +5,9 @@
   <xacro:include filename="$(find krytn)/robot_description/magni/inertial.xacro" />
   <xacro:macro name="low_friction">
-    <collision>
-      <surface>
-        <friction>
-          <mu>0.1</mu>
-          <mu1>0.1</mu1>
-          <mu2>0.1</mu2>
-          <slip1>0</slip1>
-          <slip2>0</slip2>
-        </friction>
-      </surface>
-    </collision>
+    <mu>0.1</mu>
+    <mu1>0.1</mu1>
+    <mu2>0.1</mu2>
+    <slip1>0</slip1>
+    <slip2>0</slip2>
   </xacro:macro>
   <xacro:macro name="high_friction">
@@ -27,4 +21,6 @@
             <slip1>0.0</slip1>
             <slip2>0.0</slip2>
+            <min_depth>0.001</min_depth>
+            <kp>1e8</kp>
           </ode>
         </friction>
